File: kicad/main_board/main_board.kicad_pcb (KiCad board)
At the start: 2 copper layers, 59.5 x 8 mm, 31 parts, among them J1 mic+, J2 mic-, J3 XLR2, J4 XLR1, J5 XLR3, Q1 BC859C, Q2 BC859C, Q3 BC859C, Q4 BC849C

Commit message: new R labeling, capsule pwr 2.2k
Parts:
- R9: renamed from R7; value 10k -> 2.2k
- renumbered R8 to R7, R9 to R8

Commit message: small updates and new readme
Parts:
- D1: value 10V -> 9.1V
- R4: value 33k -> 10k
- renumbered R9 to R7, R7 to R8, R8 to R9
Other:
- board text added: "diy_mm"
- board text removed: "(c)hf"
Changed lines of the file:
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@@
     (property "Sheetname" "")
     (attr smd)
-    (fp_text reference "R9" (at 0 0 180) (layer "B.SilkS")
+    (fp_text reference "R7" (at 0 0 180) (layer "B.SilkS")
       (effects (font (size 1 1) (thickness 0.15)) (justify mirror))
     )
@@
       (effects (font (size 1 1) (thickness 0.15)) (justify mirror))
     )
-    (fp_text value "10V" (at 0 -1.75 90) (layer "B.Fab")
+    (fp_text value "9.1V" (at 0 -1.75 90) (layer "B.Fab")
       (effects (font (size 1 1) (thickness 0.15)) (justify mirror))
     )
@@
       (effects (font (size 1 1) (thickness 0.15)) (justify mirror))
     )
-    (fp_text value "33k" (at 0 -1.82) (layer "B.Fab")
+    (fp_text value "10k" (at 0 -1.82) (layer "B.Fab")
       (effects (font (size 1 1) (thickness 0.15)) (justify mirror))
     )
@@
     (property "Sheetname" "")
     (attr smd)
-    (fp_text reference "R8" (at 0 0 180) (layer "B.SilkS")
+    (fp_text reference "R9" (at 0 0 180) (layer "B.SilkS")
       (effects (font (size 1 1) (thickness 0.15)) (justify mirror))
     )
@@
     (property "Sheetname" "")
     (attr smd)
-    (fp_text reference "R7" (at 0 0 90) (layer "B.SilkS")
+    (fp_text reference "R8" (at 0 0 90) (layer "B.SilkS")
       (effects (font (size 1 1) (thickness 0.15)) (justify mirror))
     )
@@
     (effects (font (size 1 1) (thickness 0.15)) (justify mirror))
   )
-  (gr_text "(c)hf" (at 157 106.5) (layer "B.SilkS")
+  (gr_text "diy_mm" (at 156 106.5) (layer "B.SilkS")
     (effects (font (size 1 1) (thickness 0.15)) (justify mirror))
   )
